Commit message: fix EoE position to grip position

File: open_manipulator_6dof_description/urdf/open_manipulator_6dof.urdf.xacro (robot description, xacro)
@@ -330,7 +330,7 @@
   <!--  Gripper joint -->
   <joint name="gripper" type="prismatic">
-    <parent link="link7"/>
+    <parent link="end_effector_link"/>
     <child link="gripper_link"/>
-    <origin xyz="0.0 0.021 0.0707" rpy="0 0 0"/>
+    <origin xyz="0.0 0.021 -0.0443" rpy="0 0 0"/>
     <axis xyz="0 1 0"/>
     <limit velocity="4.8" effort="1" lower="-0.010" upper="0.019" />
@@ -370,7 +370,7 @@
   <!--  Gripper joint sub -->
   <joint name="gripper_sub" type="prismatic">
-    <parent link="link7"/>
+    <parent link="end_effector_link"/>
     <child link="gripper_link_sub"/>
-    <origin xyz="0.0 -0.021 0.0707" rpy="0 0 0"/>
+    <origin xyz="0.0 -0.021 -0.0443" rpy="0 0 0"/>
     <axis xyz="0 -1 0"/>
     <limit velocity="4.8" effort="1" lower="-0.010" upper="0.019" />
